Commit message: Added mover4 arm macro to urdf

File: robot_description/urdf/macros.xacro (robot description, xacro)
@@ -1,4 +1,4 @@
 <?xml version="1.0"?>
-<robot name="macros" xmlns:xacro="http://ros.org/wiki/xacro">
+<robot name="macros" xmlns:xacro="http://www.ros.org/wiki/xacro">
 <!-- Common macros file for Robco robot URDF.XACRO's -->
 <!-- Created by Stefan -->

File: robot_description/urdf/materials.xacro (robot description, xacro)
@@ -1,4 +1,4 @@
 <?xml version="1.0"?>
-<robot name="materials" xmlns:xacro="http://ros.org/wiki/xacro">
+<robot name="materials" xmlns:xacro="http://www.ros.org/wiki/xacro">
 <!-- Common materials file for Robco robot URDF.XACRO's -->
 <!-- Created by Stefan -->

File: robot_description/urdf/new_base.urdf.xacro (robot description, xacro)
@@ -10,354 +10,10 @@
   <!-- 3D Sensors -->
   <!--<xacro:include filename="$(find robot_description)/urdf/kinect.urdf.xacro"/>-->
-  <!-- base_footprint is a fictitious link(frame) that is on the ground right below base_link origin, navigation stack depends on this frame -->
-<link name="base_footprint">
-  <!--base link should not have inertia!!!because of moveit and gazebo!-->
-  <!--
-    <inertial>
-      <mass value="0.0001" />
-      <origin xyz="0 0 0" />
-      <inertia ixx="0.0001" ixy="0.0" ixz="0.0"
-              iyy="0.0001" iyz="0.0"
-              izz="0.0001" />
-    </inertial>
-    -->
-    <visual>
-      <origin xyz="0 0 0" rpy="0 0 0" />
-      <geometry>
-        <box size="0.001 0.001 0.001" />
-      </geometry>
-      <material name="red" />
-    </visual>
-    <collision>
-      <origin xyz="0 0 0.017" rpy="0 0 0" />
-      <geometry>
-       <box size="0.001 0.001 0.001" />
-      </geometry>
-    </collision>
-</link>
-    <gazebo reference="base_footprint">
-        <turnGravityOff>false</turnGravityOff>
-    </gazebo>
-  <!-- JOINT BASE_LINK TO BASE_FRAME-->
-  <joint name="base_footprint_base_link_joint" type="fixed">
-    <origin rpy="0 0 0" xyz="0 0 ${base_from_base_frame_Z_offset}"/>
-    <parent link="base_footprint"/>
-    <child link="base_link"/>
-  </joint>
-<!-- BASE-LINK -->
-  <!--Center on the bottom side of the base plate of the robot-->
- <link name="base_link">
-   <pose>0 0 0.1 0 0 0</pose>
-   <inertial>
-      <origin xyz="0.0 0 ${eddie_plate_half_height}" rpy=" 0 0 0"/>
-      <mass value="${base_mass}"/>
-      <inertia
-          ixx="0.1" ixy="0" ixz="0"
-          iyy="0.1" iyz="0"
-          izz="0.1"
-      />
-    </inertial>
-    <collision name="collision">
-    <origin xyz="0 0 ${eddie_plate_half_height}" rpy="0 0 0" />
-      <geometry>
-       <cylinder radius="${eddie_plate_radius}" length="${eddie_plate_height}"/>
-      </geometry>
-    </collision>
-    <visual name="base_visual">
-      <!--<origin xyz="0 0 ${eddie_plate_half_height}" rpy="0 0 0" />      -->
-      <origin xyz="0 0 0" rpy="${ROTATE_90_DEGREES} 0 ${ROTATE_90_DEGREES}"/>
-      <geometry>
-        <!--<cylinder radius="${eddie_plate_radius}" length="${eddie_plate_height}"/>-->
-        <mesh filename="package://robot_description/meshes/Eddiebot/ArloBottomplateTST.dae" scale="0.001 0.001 0.001"/>
-      </geometry>
-      <!--<material name="orange"/>-->
-    </visual>
-  </link>
-<!--###########  DRIVE WHEELS #############################-->
-<!--########### left wheel #############################-->
-  <link name="left_wheel">
-    <collision name="collision">
-      <origin xyz="0 0 0" rpy="0 ${ROTATE_90_DEGREES} ${ROTATE_90_DEGREES}"/>
-      <geometry>
-        <cylinder radius="${wheel_radius}" length="${wheel_width}"/>
-      </geometry>
-    </collision>
-    <visual name="left_wheel_visual">
-      <!--<origin xyz="0 0 0" rpy="0 1.5707 1.5707"/>-->
-      <origin xyz="0 0 0" rpy="0 ${2*ROTATE_90_DEGREES} ${ROTATE_90_DEGREES}"/>
-      <geometry>
-        <mesh filename="package://robot_description/meshes/Eddiebot/wheel.dae" scale="0.0012 0.0012 0.0012"/>
-        <!--<cylinder radius="${wheel_radius}" length="${wheel_width}"/>-->
-      </geometry>
-    </visual>
-    <inertial>
-      <origin xyz="0 0 0" rpy="0 ${ROTATE_90_DEGREES} ${ROTATE_90_DEGREES}"/>
-      <mass value="5"/>
-      <inertia
-        ixx=".1" ixy="0.0" ixz="0.0"
-        iyy=".1" iyz="0.0"
-        izz=".1"/>
-    </inertial>
-  </link>
-  <joint type="continuous" name="left_wheel_hinge">
-    <origin xyz="0 ${base_y_origin_to_wheel_origin} ${base_z_origin_to_wheel_origin}" rpy="0 0 0"/>
-        <!--<origin xyz="0 0.19 -${0.10 - 0.0231}" rpy="0 0 0"/>-->
-    <child link="left_wheel"/>
-    <parent link="base_link"/>
-    <axis xyz="0 1 0" rpy="0 0 0"/>
-    <limit effort="10000" velocity="1000"/>
-    <joint_properties damping="1.0" friction="1.0"/>
-  </joint>
-<!--########### right wheel #############################-->
-  <link name="right_wheel">
-    <collision name="collision">
-      <origin xyz="0 0 0" rpy="0 ${ROTATE_90_DEGREES} ${ROTATE_90_DEGREES}"/>
-      <geometry>
-        <cylinder radius="${wheel_radius}" length="${wheel_width}"/>
-      </geometry>
-    </collision>
-    <visual name="left_wheel_visual">
-      <!--<origin xyz="0 0 0" rpy="0 1.5707 1.5707"/>-->
-      <origin xyz="0 0 0" rpy="0 0 ${ROTATE_90_DEGREES}"/>
-      <geometry>
-        <mesh filename="package://robot_description/meshes/Eddiebot/wheel.dae" scale="0.0012 0.0012 0.0012"/>
-        <!--<cylinder radius="${wheel_radius}" length="${wheel_width}"/>-->
-      </geometry>
-    </visual>
-    <inertial>
-      <origin xyz="0 0 0" rpy="0 ${ROTATE_90_DEGREES} ${ROTATE_90_DEGREES}"/>
-      <mass value="5"/>
-      <inertia
-        ixx=".1" ixy="0.0" ixz="0.0"
-        iyy=".1" iyz="0.0"
-        izz=".1"/>
-    </inertial>
-  </link>
-  <joint type="continuous" name="right_wheel_hinge">
-    <origin xyz="0 -${base_y_origin_to_wheel_origin} ${base_z_origin_to_wheel_origin}" rpy="0 0 0"/>
-    <!--<origin xyz="0 -0.19 -0.0231" rpy="0 0 0"/>-->
-    <child link="right_wheel"/>
-    <parent link="base_link"/>
-    <axis xyz="0 1 0" rpy="0 0 0"/>
-    <limit effort="10000" velocity="1000"/>
-    <joint_properties damping="1.0" friction="1.0"/>
-  </joint>
-<!--########################################-->
-<!--###########  CASTER WHEELS #############################-->
-<!--########### caster front #############################-->
-  <link name="caster_box_front">
-    <collision name="collision">
-      <origin xyz="0 0 0" rpy="0 0 0"/>
-      <geometry>
-        <box size="${caster_box_lenght/2} ${caster_box_width/2} ${caster_box_height}"/>
-      </geometry>
-    </collision>
-    <!--NO VISUAL FOR NOW    ->       TODO: CREATE MESH FOR THE CASTER WHEEL-->
-    <!--<visual name="caster_box_front_visual">
-      <origin xyz="0 0 0" rpy="0 0 0"/>
-      <geometry>
-        <box size="${caster_box_lenght/2} ${caster_box_width/2} ${caster_box_height}"/>
-      </geometry>
-       <material name="black"/>
-    </visual>-->
-    <inertial>
-      <origin xyz="0 0 0" rpy="0 0 0"/>
-      <mass value="0.15"/>
-      <inertia
-        ixx=".1" ixy="0.0" ixz="0.0"
-        iyy=".1" iyz="0.0"
-        izz=".1"/>
-    </inertial>
-  </link>
-    <!-- JOINT caster_box_front TO base_link-->
-  <joint name="base_caster_box_front_joint" type="fixed">
-    <!-- NB: Z goes to - as we are below bottom deck(base) -->
-    <origin rpy="0 0 0" xyz="${caster_X_offset_from_base_link} 0 -${caster_box_height/2}"/>
-    <parent link="base_link"/>
-    <child link="caster_box_front"/>
-  </joint>
-     <!--********caster sphere front*********************-->
-    <link name="caster_sphere_front">
-        <collision name="collision">
-            <origin xyz="0 0 0" rpy="0 0 0"/>
-            <geometry>
-                <sphere radius="${caster_sphere_radius}"/>
-            </geometry>
-        </collision>
-        <!--NO VISUAL FOR NOW    ->       TODO: CREATE MESH FOR THE CASTER WHEEL-->
-        <!--<visual name="caster_sphere_front_visual">
-      <origin xyz="0 0 0" rpy="0 0 0"/>
-      <geometry>
-        <sphere radius="${caster_sphere_radius}"/>
-      </geometry>
-      <material name="black"/>
-        </visual>-->
-        <inertial>
-      <origin xyz="0 0 0" rpy="0 0 0"/>
-      <mass value="0.15"/>
-      <inertia
-        ixx=".1" ixy="0.0" ixz="0.0"
-        iyy=".1" iyz="0.0"
-        izz=".1"/>
-        </inertial>
-    </link>
-    <!-- JOINT caster_sphere_front TO caster_box_front-->
-  <joint name="caster_box_front_caster_sphere_front_joint" type="fixed">
-    <!-- NB: Z goes to - as we are below bottom deck(base)-->
-    <origin rpy="0 0 0" xyz="0 0 -${caster_box_height/2 + caster_sphere_radius}"/>
-    <parent link="caster_box_front"/>
-    <child link="caster_sphere_front"/>
-  </joint>
-<!--########### caster back #############################-->
-  <link name="caster_box_back">
-    <collision name="collision">
-      <origin xyz="0 0 0" rpy="0 0 0"/>
-      <geometry>
-        <box size="${caster_box_lenght/2} ${caster_box_width/2} ${caster_box_height}"/>
-      </geometry>
-    </collision>
-    <!--NO VISUAL FOR NOW    ->       TODO: CREATE MESH FOR THE CASTER WHEEL-->
-    <!--<visual name="caster_box_front_visual">
-      <origin xyz="0 0 0" rpy="0 0 0"/>
-      <geometry>
-        <box size="${caster_box_lenght/2} ${caster_box_width/2} ${caster_box_height}"/>
-      </geometry>
-       <material name="black"/>
-    </visual>-->
-    <inertial>
-      <origin xyz="0 0 0" rpy="0 0 0"/>
-      <mass value="0.15"/>
-      <inertia
-        ixx=".1" ixy="0.0" ixz="0.0"
-        iyy=".1" iyz="0.0"
-        izz=".1"/>
-    </inertial>
-  </link>
-    <!-- JOINT caster_box_back TO base_link-->
-  <joint name="base_caster_box_back_joint" type="fixed">
-     <!-- NB: Z goes to - as we are below bottom deck(base) -->
-    <origin rpy="0 0 0" xyz="-${caster_X_offset_from_base_link} 0 -${caster_box_height/2}"/>
-    <parent link="base_link"/>
-    <child link="caster_box_back"/>
-  </joint>
-     <!--*********caster sphere back********************-->
-    <link name="caster_sphere_back">
-        <collision name="collision">
-            <origin xyz="0 0 0" rpy="0 0 0"/>
-            <geometry>
-            <sphere radius="${caster_sphere_radius}"/>
-            </geometry>
-        </collision>
-        <!--NO VISUAL FOR NOW    ->       TODO: CREATE MESH FOR THE CASTER WHEEL-->
-        <!--<visual name="caster_sphere_front_visual">
-            <origin xyz="0 0 0" rpy="0 0 0"/>
-            <geometry>
-                <sphere radius="${caster_sphere_radius}"/>
-            </geometry>
-            <material name="black"/>
-        </visual>-->
-        <inertial>
-            <origin xyz="0 0 0" rpy="0 0 0"/>
-            <mass value="0.15"/>
-            <inertia
-                ixx=".1" ixy="0.0" ixz="0.0"
-                iyy=".1" iyz="0.0"
-                izz=".1"/>
-        </inertial>
-    </link>
-    <!-- JOINT caster_sphere_back TO caster_box_back-->
-  <joint name="caster_box_back_caster_sphere_back_joint" type="fixed">
-    <!-- NB: Z goes to - as we are below bottom deck(base)-->
-    <origin rpy="0 0 0" xyz="0 0 -${caster_box_height/2 + caster_sphere_radius}"/>
-    <parent link="caster_box_back"/>
-    <child link="caster_sphere_back"/>
-  </joint>
-<!--########################################-->
-<!--###########  STANDOFFS ON BASE PLATE  #############################-->
-  <robco_standoff_first_second_deck parent="base_link" number="0" lenght= "${top_first_botom_second_deck_distance}" x_loc="0.09" y_loc="0.165" z_loc="${eddie_plate_height}"/>
-  <robco_standoff_first_second_deck parent="base_link" number="1" lenght= "${top_first_botom_second_deck_distance}" x_loc="0.09" y_loc="-0.165" z_loc="${eddie_plate_height}"/>
-  <robco_standoff_first_second_deck parent="base_link" number="2" lenght= "${top_first_botom_second_deck_distance}" x_loc="-0.09" y_loc="0.165" z_loc="${eddie_plate_height}"/>
-  <robco_standoff_first_second_deck parent="base_link" number="3" lenght= "${top_first_botom_second_deck_distance}" x_loc="-0.09" y_loc="-0.165" z_loc="${eddie_plate_height}"/>
-<!--########################################-->
-<!--###########  SECOND DECK  #############################-->
- <!-- JOINT second_deck TO BASE_LINK -->
-  <joint name="base_link_second_deck_joint" type="fixed">
-    <origin rpy="0 0 0" xyz="0 0 ${second_deck_from_base_link_Z_offset+eddie_plate_half_height}"/>
-    <parent link="base_link"/>
-    <child link="second_deck"/>
-  </joint>
-  <!--Link centered on the bottom side of the second deck/plate of the robot-->
-  <link name="second_deck">
-    <pose>0 0 0.1 0 0 0</pose>
-    <inertial>
-      <mass value="${second_deck_mass}"/>
-      <origin xyz="0.0 0 0" rpy=" 0 0 0"/>
-      <inertia
-          ixx="0.1" ixy="0" ixz="0"
-          iyy="0.1" iyz="0"
-          izz="0.1"
-      />
-    </inertial>
-    <collision name="collision">
-        <origin xyz="0 0 ${eddie_plate_half_height}" rpy="0 0 0" />
-      <geometry>
-       <cylinder radius="${eddie_plate_radius}" length="${eddie_plate_height}"/>
-      </geometry>
-    </collision>
-    <visual name="second_deck_visual">
-        <!--<origin xyz="0 0 ${eddie_plate_half_height}" rpy="0 0 0" />      -->
-      <origin xyz="0 0 0" rpy="${ROTATE_90_DEGREES} 0 ${ROTATE_90_DEGREES}"/>
-      <geometry>
-        <!--<cylinder radius="${eddie_plate_radius}" length="${eddie_plate_height}"/>-->
-        <mesh filename="package://robot_description/meshes/Eddiebot/ArloBottomplateTST.dae" scale="0.001 0.001 0.001"/>
-      </geometry>
-      <material name="orange"/>
-    </visual>
-  </link>
-<!--########################################-->
-<!--###########  STANDOFFS ON SECOND PLATE  #############################-->
-  <robco_standoff_first_second_deck parent="second_deck" number="0" lenght= "${top_first_botom_second_deck_distance}" x_loc="0.09" y_loc="0.165" z_loc="${eddie_plate_height}"/>
-  <robco_standoff_second_third_deck parent="second_deck" number="1" lenght= "${top_second_botom_third_deck_distance}" x_loc="0.09" y_loc="-0.165" z_loc="${eddie_plate_height}"/>
-  <robco_standoff_second_third_deck parent="second_deck" number="2" lenght= "${top_second_botom_third_deck_distance}" x_loc="-0.09" y_loc="0.165" z_loc="${eddie_plate_height}"/>
-  <robco_standoff_second_third_deck parent="second_deck" number="3" lenght= "${top_second_botom_third_deck_distance}" x_loc="-0.09" y_loc="-0.165" z_loc="${eddie_plate_height}"/>
-<!--########################################-->
-<!--######### THIRD DECK ###############################-->
-  <!-- JOINT THIRD_DECK TO SECOND_DECK -->
-  <joint name="third_deck_second_deck_joint" type="fixed">
-    <origin rpy="0 0 0" xyz="0 0 ${third_deck_from_second_deck_Z_offset+eddie_plate_half_height}"/>
-    <parent link="second_deck"/>
-    <child link="third_deck"/>
-  </joint>
-  <!--Link centered on the bottom side of the third plate of the robot-->
-  <link name="third_deck">
-    <pose>0 0 0.1 0 0 0</pose>
-    <inertial>
-      <mass value="${third_deck_mass}"/>
-      <origin xyz="0.0 0 0.1" rpy=" 0 0 0"/>
-      <inertia
-          ixx="0.1" ixy="0" ixz="0"
-          iyy="0.1" iyz="0"
-          izz="0.1"
-      />
-    </inertial>
-    <collision name="collision">
-      <origin xyz="0 0 ${eddie_plate_half_height}" rpy="0 0 0" />
-      <geometry>
-       <cylinder radius="${eddie_plate_radius}" length="${eddie_plate_height}"/>
-      </geometry>
-    </collision>
-    <visual name="third_deck__visual">
-      <origin xyz="0 0 0" rpy="${ROTATE_90_DEGREES} 0 ${ROTATE_90_DEGREES}"/>
-      <geometry>
-        <!--<cylinder radius="${base_radius}" length="${base_height}"/>-->
-        <mesh filename="package://robot_description/meshes/Eddiebot/ArloBottomplateTST.dae" scale="0.001 0.001 0.001"/>
-      </geometry>
-      <material name="orange"/>
-    </visual>
-  </link>
-<!--########################################-->
-<!--###########  KINECT STANDOFFS ON THIRD PLATE  #############################-->
-  <robco_standoff_first_second_deck parent="second_deck" number="0" lenght= "${top_first_botom_second_deck_distance}" x_loc="0.09" y_loc="0.165" z_loc="${eddie_plate_height}"/>
-  <robco_standoff_second_third_deck parent="second_deck" number="1" lenght= "${top_second_botom_third_deck_distance}" x_loc="0.09" y_loc="-0.165" z_loc="${eddie_plate_height}"/>
+   <xacro:include filename="$(find robot_description)/urdf/new_mover4.macro.urdf.xacro" />
+<!--###################################################################################-->
+<!--###################################################################################-->
+<!--###################################################################################-->
+<!--###################################################################################-->
+<!--###################################################################################-->
 <!--###################################################################################-->
 <!-- ####### generic constants ##### -->
@@ -396,4 +52,5 @@
   <xacro:property name="third_deck_radius" value="${17.75*SCALE_in_m/2}" />
   <xacro:property name="third_deck_mass" value="1.5" />   <!-- in kg -->
+<!--Base height to top of third deck = 42.775 cm ???-->
   <!-- Wheels -->
   <xacro:property name="wheel_diameter" value="${6*SCALE_in_m}" />
@@ -421,24 +78,35 @@
  <!-- Kinect -->
  <!-- kinect_mount_point - joint data for maunting kinect relative to base_link  -->
-  <xacro:property name="kinect_mount_point_from_base_link_Z_offset" value="0.50" />
-  <!--<xacro:property name="kinect_mount_point_from_base_link_X_offset" value="-${base_radius - 0.10}"/> -->
-  <xacro:property name="kinect_mount_point_from_base_link_X_offset" value="-${0.14509}"/>
-  <xacro:property name="kinect_support_height" value="0.02" />
-  <xacro:property name="kinect_support_width" value="${eddie_plate_height}" />
-  <xacro:property name="kinect_support_lenght" value="0.02" />
-  <xacro:property name="kinect_support_mass" value=".05" />    <!--in kg-->
+ <!--Kinect mount height 50 cm fro ground ?????-->
+    <xacro:property name="kinect_standoff_lenght" value="${0.42775}" />
+    <xacro:property name="kinect_standoff_X_offset" value="${-0.15}" />
+    <xacro:property name="kinect_standoff_Y_offset" value="${0.06}" />
+    <xacro:property name="kinect_standoff_Z_offset" value="${eddie_plate_height}" />
+  <!--<xacro:property name="kinect_mount_point_from_kinect_standoff_0__Z_offset" value="${(kinect_standoff_lenght - eddie_plate_height)/2+eddie_plate_height}" />
+  <xacro:property name="kinect_mount_point_from_kinect_standoff_0__X_offset" value="${0.15}"/>-->
+  <xacro:property name="kinect_mount_point_from_support_plate_X_offset" value="${0.0}"/>
+  <xacro:property name="kinect_mount_point_from_support_plate_Y_offset" value="${0.0}" />
+  <xacro:property name="kinect_mount_point_from_support_plate_Z_offset" value="${eddie_plate_half_height}" />
+  <xacro:property name="kinect_support_from_kinect_standoff_0__X_offset" value="${0.0}"/>
+  <xacro:property name="kinect_support_from_kinect_standoff_0__Y_offset" value="${-0.06}"/>
+  <xacro:property name="kinect_support_from_kinect_standoff_0__Z_offset" value="${(kinect_standoff_lenght - eddie_plate_height)/2+eddie_plate_half_height}" />
+  <xacro:property name="kinect_support_height" value="${eddie_plate_height}" />
+  <xacro:property name="kinect_support_width" value="${0.15}" />
+  <xacro:property name="kinect_support_lenght" value="${0.06}" />
+  <xacro:property name="kinect_support_mass" value="${.05}" />    <!--in kg-->
   <!-- Hokuyo Laser scanner -->
-  <xacro:property name="hokuyo_size" value="0.05" />
+  <xacro:property name="hokuyo_size" value="${0.05}" />
     <!-- camera -->
-  <xacro:property name="cameraSize" value="0.05"/>
-  <xacro:property name="cameraMass" value="0.1"/>
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
File: robot_description/urdf/new_gazebo.urdf.xacro (robot description, xacro)
@@ -1,7 +1,7 @@
 <?xml version="1.0"?>
-<robot xmlns:controller="http://playerstage.sourceforge.net/gazebo/xmlschema/#controller" xmlns:interface="http://playerstage.sourceforge.net/gazebo/xmlschema/#interface" xmlns:sensor="http://playerstage.sourceforge.net/gazebo/xmlschema/#sensor" xmlns:xacro="http://ros.org/wiki/xacro" name="eddiebot_gazebo">
+<robot xmlns:controller="http://playerstage.sourceforge.net/gazebo/xmlschema/#controller" xmlns:interface="http://playerstage.sourceforge.net/gazebo/xmlschema/#interface" xmlns:sensor="http://playerstage.sourceforge.net/gazebo/xmlschema/#sensor" xmlns:xacro="http://ros.org/wiki/xacro" name="robco_gazebo">
 <!-- ASUS Xtion PRO camera for simulation -->
 <!-- gazebo_ros_wge100 plugin is in kt2_gazebo_plugins package -->
-<xacro:macro name="eddiebot_sim_asus_xtion">
+<xacro:macro name="robco_sim_asus_xtion">
   <gazebo reference="camera_link" >
     <sensor:camera name="camera" >
@@ -32,5 +32,5 @@
   </gazebo>
 </xacro:macro>
-<xacro:macro name="eddiebot_sim_kinect">
+<xacro:macro name="robco_sim_kinect">
   <gazebo reference="camera_link">
     <sensor:camera name="camera">
@@ -58,5 +58,5 @@
   </gazebo>
 </xacro:macro>
-<xacro:macro name="eddiebot_sim_imu">
+<xacro:macro name="robco_sim_imu">
   <gazebo>
     <controller:gazebo_ros_imu name="imu_controller" plugin="libgazebo_ros_imu.so">
@@ -72,5 +72,5 @@
   </gazebo>
 </xacro:macro>
-<xacro:macro name="eddiebot_sim_laser">
+<xacro:macro name="robco_sim_laser">
   <gazebo reference="laser">
     <sensor:ray name="laser">
@@ -97,9 +97,9 @@
   </gazebo>
 </xacro:macro>
-<xacro:macro name="eddiebot_sim_create">
+<xacro:macro name="robco_sim_create">
   <gazebo>
     <controller:gazebo_ros_create name="create_controller" plugin="libgazebo_ros_create.so">
       <alwaysOn>true</alwaysOn>
-      <node_namespace>eddiebot_node</node_namespace>
+      <node_namespace>robco_node</node_namespace>
       <left_wheel_joint>left_wheel_joint</left_wheel_joint>
       <right_wheel_joint>right_wheel_joint</right_wheel_joint>
@@ -114,5 +114,5 @@
   </gazebo>
 </xacro:macro>
-<xacro:macro name="eddiebot_sim_wall_sensors">
+<xacro:macro name="robco_sim_wall_sensors">
   <gazebo reference="wall_sensor_link">
     <sensor:ray name="wall_sensor">
