Commit message: Added mover4 arm macro to urdf

File: robot_description/urdf/new_kinect.urdf.xacro (robot description, xacro)
@@ -1,12 +1,12 @@
 <?xml version="1.0"?>
-<robot name="eddiebot_hardware" xmlns:xacro="http://ros.org/wiki/xacro">
+<robot name="robco_hardware" xmlns:xacro="http://ros.org/wiki/xacro">
   <property name="M_PI" value="3.14159"/>
-  <include filename="$(find eddiebot_description)/urdf/gazebo.urdf.xacro"/>
-  <include filename="$(find eddiebot_description)/urdf/eddiebot_calibration.xacro" />
-<xacro:macro name="eddiebot_kinect">
+  <include filename="$(find robco_description)/urdf/new_gazebo.urdf.xacro"/>
+  <include filename="$(find robco_description)/urdf/new_calibration.xacro" />
+<xacro:macro name="robco_kinect">
   <joint name="base_camera_joint" type="fixed">
-    <origin xyz="${eddiebot_calib_cam_x} ${eddiebot_calib_cam_y} ${eddiebot_calib_cam_z}"
-            rpy="${eddiebot_calib_cam_rr} ${eddiebot_calib_cam_rp} ${eddiebot_calib_cam_ry}" />
-    <parent link="${eddiebot_camera_parent_name}" />
+    <origin xyz="${robco_calib_cam_x} ${robco_calib_cam_y} ${robco_calib_cam_z}"
+            rpy="${robco_calib_cam_rr} ${robco_calib_cam_rp} ${robco_calib_cam_ry}" />
+    <parent link="${robco_camera_parent_name}" />
     <child link="camera_link" />
   </joint>
@@ -22,5 +22,5 @@
       <origin xyz=" 0 0 0 " rpy="0 0 0" />
       <geometry>
-        <mesh filename="package://eddiebot_description/meshes/kinect.dae"/>
+        <mesh filename="package://robot_description/meshes/kinect.dae"/>
       </geometry>
     </visual>
@@ -89,5 +89,5 @@
   </link>
   <!-- Kinect sensor for simulation -->
-  <eddiebot_sim_kinect/>
+  <new_sim_kinect/>
 </xacro:macro>
 </robot>

File: robot_description/urdf/new_properties.xacro (robot description, xacro)
@@ -33,3 +33,33 @@
   <xacro:property name="third_deck_radius" value="${17.75*SCALE_in_m/2}" />
   <xacro:property name="third_deck_mass" value="1.5" />   <!-- in kg -->
+ <xacro:macro name="robco_kinect_support_plate" params="parent lenght width height x_loc y_loc z_loc">
+    <joint name="standoff_kinect_support_plate_joint" type="fixed">
+      <origin xyz="${x_loc} ${y_loc} ${z_loc+lenght/2}" rpy="0 0 0" />
+      <parent link="${parent}"/>
+      <child link="standoff_kinect_support_plate_link" />
+    </joint>
+    <link name="standoff_kinect_support_plate_link">
+      <inertial>
+        <mass value="0.001" />
+        <origin xyz="0 0 0" />
+        <inertia ixx="0.0001" ixy="0.0" ixz="0.0"
+          iyy="0.0001" iyz="0.0"
+          izz="0.0001" />
+      </inertial>
+      <visual>
+        <origin xyz=" 0 0 0 " rpy="0 0 0" />
+        <geometry>
+        <box size="${lenght} ${width} ${height}"/>
+          <!--<mesh filename="package://robot_description/meshes/68-02421-8000-RA_Eddiebot_F-F_Standoff.dae" scale="${SCALE_mm_m} ${SCALE_mm_m} ${SCALE_mm_m}"/>-->
+        </geometry>
+        <material name="black"/>
+      </visual>
+      <collision>
+        <origin xyz="0.0 0.0 0.0" rpy="0 0 0" />
+        <geometry>
+        <box size="${lenght} ${width} ${height}"/>
+        </geometry>
+      </collision>
+    </link>
+  </xacro:macro>
 </robot>
