Commit message: urdf kinect  and dimension changes

File: robot_description/urdf/new_base.urdf.xacro (robot description, xacro)
@@ -19,4 +19,5 @@
 <!-- ####### generic constants ##### -->
   <!--All units in m-kg-s-radians unit system -->
+  <xacro:property name="PI" value="3.1415" />
   <xacro:property name="M_PI" value="3.14159265358979323846264338327950288419716" />
   <!--<xacro:property name="M_PI" value="3.1415926535897931" />-->
@@ -87,12 +88,22 @@
   <xacro:property name="kinect_mount_point_from_support_plate_X_offset" value="${0.0}"/>
   <xacro:property name="kinect_mount_point_from_support_plate_Y_offset" value="${0.0}" />
-  <xacro:property name="kinect_mount_point_from_support_plate_Z_offset" value="${eddie_plate_half_height}" />
+  <xacro:property name="kinect_mount_point_from_support_plate_Z_offset" value="${kinect_support_half_height}" />
   <xacro:property name="kinect_support_from_kinect_standoff_0__X_offset" value="${0.0}"/>
   <xacro:property name="kinect_support_from_kinect_standoff_0__Y_offset" value="${-0.06}"/>
-  <xacro:property name="kinect_support_from_kinect_standoff_0__Z_offset" value="${(kinect_standoff_lenght - eddie_plate_height)/2+eddie_plate_half_height}" />
+  <xacro:property name="kinect_support_from_kinect_standoff_0__Z_offset" value="${(kinect_standoff_lenght - kinect_support_height)/2+kinect_support_half_height}" />
   <xacro:property name="kinect_support_height" value="${eddie_plate_height}" />
+  <xacro:property name="kinect_support_half_height" value="${kinect_support_height/2}" />
   <xacro:property name="kinect_support_width" value="${0.15}" />
   <xacro:property name="kinect_support_lenght" value="${0.06}" />
   <xacro:property name="kinect_support_mass" value="${.05}" />    <!--in kg-->
+    <!-- Define a Kinect dimensions using properties -->
+   <xacro:property name="kinect_body_x" value="0.07271" />
+   <xacro:property name="kinect_body_y" value="0.27794" />
+   <xacro:property name="kinect_body_z" value="0.033" />
+   <xacro:property name="kinect_base_x" value="0.072" />
+   <xacro:property name="kinect_base_y" value="0.085" />
+   <xacro:property name="kinect_base_z" value="0.021" />
+   <xacro:property name="kinect_base_post_height" value="0.016" />
+   <xacro:property name="kinect_base_post_radius" value="0.005" />
   <!-- Hokuyo Laser scanner -->
   <xacro:property name="hokuyo_size" value="${0.05}" />
@@ -280,4 +291,126 @@
     </link>
   </xacro:macro>
+<!--######################  KINECT MACRO  #############################################################-->
+<!--https://github.com/pirobot/rbx2/blob/indigo-devel/rbx2_description/urdf/box_robot/box_robot_with_kinect.xacro-->
+ <!-- Define a box-shaped camera link for the Kinect -->
+   <xacro:macro name="kinect_camera" params="parent name color *origin">
+      <joint name="${parent}_${name}_joint" type="fixed">
+         <xacro:insert_block name="origin" />
+         <parent link="${parent}_link"/>
+         <child link="${name}_base_link"/>
+      </joint>
+      <link name="${name}_base_link">
+         <visual>
+            <origin xyz="0 0.0 0.0" rpy="0 0 0" />
+            <geometry>
+               <box size="${kinect_base_x} ${kinect_base_y} ${kinect_base_z}"/>
+            </geometry>
+            <material name="${color}" />
+         </visual>
+         <collision>
+            <origin xyz="0 0 0" rpy="0 0 0" />
+            <geometry>
+               <box size="${kinect_base_x} ${kinect_base_y} ${kinect_base_z}"/>
+            </geometry>
+         </collision>
+      </link>
+      <joint name="${name}_base_post_joint" type="fixed">
+         <origin xyz="0 0 ${(kinect_base_z + kinect_base_post_height)/2}" rpy="0 0 0" />
+         <parent link="${name}_base_link" />
+         <child link="${name}_base_post_link" />
+      </joint>
+      <link name="${name}_base_post_link">
+         <visual>
+            <origin xyz="0 0 0" rpy="0 0 0" />
+            <geometry>
+               <cylinder radius="${kinect_base_post_radius}" length="${kinect_base_post_height}"/>
+            </geometry>
+            <material name="${color}" />
+         </visual>
+         <collision>
+            <origin xyz="0 0 0" rpy="0 0 0" />
+            <geometry>
+               <cylinder radius="${kinect_base_post_radius}" length="${kinect_base_post_height}"/>
+            </geometry>
+         </collision>
+      </link>
+      <joint name="${name}_base_joint" type="fixed">
+         <origin xyz="0 0 ${(kinect_base_post_height + kinect_body_z)/2}" rpy="0 0 0" />
+         <parent link="${name}_base_post_link" />
+         <child link="${name}_link" />
+      </joint>
+      <link name="${name}_link">
+         <visual>
+            <!--<origin xyz="0 0 0" rpy="0 0 0" />-->
+            <origin xyz="0 0 0" rpy="0 0 0" />
+            <geometry>
+               <box size="${kinect_body_x} ${kinect_body_y} ${kinect_body_z}"/>
+            </geometry>
+            <material name="${color}" />
+         </visual>
+         <collision>
+            <origin xyz="0 0 0" rpy="0 0 0" />
+            <geometry>
+               <box size="${kinect_body_x} ${kinect_body_y} ${kinect_body_z}"/>
+            </geometry>
+         </collision>
+      </link>
+      <joint name="${name}_depth_joint" type="fixed">
+         <origin xyz="0 0.0125 0" rpy="0 0 0" />
+          <parent link="${name}_link" />
+          <child link="${name}_depth_frame" />
+      </joint>
+      <link name="${name}_depth_frame">
+      <inertial>
+         <mass value="0.000001" />
+         <origin xyz="0 0 0" />
+         <inertia ixx="0.0001" ixy="0.0" ixz="0.0"
+            iyy="0.0001" iyz="0.0"
+            izz="0.0001" />
+         </inertial>
+      </link>
+      <joint name="${name}_depth_optical_joint" type="fixed">
+         <origin xyz="0 0 0" rpy="${-PI/2} 0 ${-PI/2}" />
+         <parent link="${name}_depth_frame" />
+         <child link="${name}_depth_optical_frame" />
+      </joint>
+      <link name="${name}_depth_optical_frame">
+         <inertial>
+            <mass value="0.000001" />
+            <origin xyz="0 0 0" />
+            <inertia ixx="0.0001" ixy="0.0" ixz="0.0"
+               iyy="0.0001" iyz="0.0"
+               izz="0.0001" />
+         </inertial>
+      </link>
+      <joint name="${name}_rgb_joint" type="fixed">
+         <origin xyz="0 -0.0125 0" rpy="0 0 0" />
+         <parent link="${name}_link" />
+         <child link="${name}_rgb_frame" />
+      </joint>
+      <link name="${name}_rgb_frame">
+         <inertial>
+         <mass value="0.000001" />
+         <origin xyz="0 0 0" />
+         <inertia ixx="0.0001" ixy="0.0" ixz="0.0"
+            iyy="0.0001" iyz="0.0"
+            izz="0.0001" />
+         </inertial>
+      </link>
+      <joint name="${name}_rgb_optical_joint" type="fixed">
+         <origin xyz="0 0 0" rpy="${-PI/2} 0 ${-PI/2}" />
+         <parent link="${name}_rgb_frame" />
+         <child link="${name}_rgb_optical_frame" />
+      </joint>
+      <link name="${name}_rgb_optical_frame">
+         <inertial>
+            <mass value="0.000001" />
+            <origin xyz="0 0 0" />
+            <inertia ixx="0.0001" ixy="0.0" ixz="0.0"
+               iyy="0.0001" iyz="0.0"
+               izz="0.0001" />
+         </inertial>
+      </link>
+   </xacro:macro>
 <!--###################################################################################-->
 <!--###################################################################################-->
@@ -555,8 +688,8 @@
   <robco_standoff_first_second_deck parent="base_link" number="2" lenght= "${top_first_botom_second_deck_distance}" x_loc="-0.09" y_loc="0.165" z_loc="${eddie_plate_height}"/>
   <robco_standoff_first_second_deck parent="base_link" number="3" lenght= "${top_first_botom_second_deck_distance}" x_loc="-0.09" y_loc="-0.165" z_loc="${eddie_plate_height}"/>-->
-  <robco_standoff parent="base_link" subname="first_second_deck" number="0" lenght= "${top_first_botom_second_deck_distance}" x_loc="0.09" y_loc="0.165" z_loc="${eddie_plate_height}"/>
-  <robco_standoff parent="base_link" subname="first_second_deck" number="1" lenght= "${top_first_botom_second_deck_distance}" x_loc="0.09" y_loc="-0.165" z_loc="${eddie_plate_height}"/>
-  <robco_standoff parent="base_link" subname="first_second_deck" number="2" lenght= "${top_first_botom_second_deck_distance}" x_loc="-0.09" y_loc="0.165" z_loc="${eddie_plate_height}"/>
-  <robco_standoff parent="base_link" subname="first_second_deck" number="3" lenght= "${top_first_botom_second_deck_distance}" x_loc="-0.09" y_loc="-0.165" z_loc="${eddie_plate_height}"/>
+  <xacro:robco_standoff parent="base_link" subname="first_second_deck" number="0" lenght= "${top_first_botom_second_deck_distance}" x_loc="0.09" y_loc="0.165" z_loc="${eddie_plate_height}"/>
+  <xacro:robco_standoff parent="base_link" subname="first_second_deck" number="1" lenght= "${top_first_botom_second_deck_distance}" x_loc="0.09" y_loc="-0.165" z_loc="${eddie_plate_height}"/>
+  <xacro:robco_standoff parent="base_link" subname="first_second_deck" number="2" lenght= "${top_first_botom_second_deck_distance}" x_loc="-0.09" y_loc="0.165" z_loc="${eddie_plate_height}"/>
+  <xacro:robco_standoff parent="base_link" subname="first_second_deck" number="3" lenght= "${top_first_botom_second_deck_distance}" x_loc="-0.09" y_loc="-0.165" z_loc="${eddie_plate_height}"/>
 <!--########################################-->
 <!--###########  SECOND DECK  #############################-->
@@ -601,8 +734,8 @@
   <robco_standoff_second_third_deck parent="second_deck" number="2" lenght= "${top_second_botom_third_deck_distance}" x_loc="-0.09" y_loc="0.165" z_loc="${eddie_plate_height}"/>
   <robco_standoff_second_third_deck parent="second_deck" number="3" lenght= "${top_second_botom_third_deck_distance}" x_loc="-0.09" y_loc="-0.165" z_loc="${eddie_plate_height}"/>-->
-  <robco_standoff parent="second_deck" subname="second_third_deck" number="0" lenght= "${top_first_botom_second_deck_distance}" x_loc="0.09" y_loc="0.165" z_loc="${eddie_plate_height}"/>
-  <robco_standoff parent="second_deck" subname="second_third_deck" number="1" lenght= "${top_second_botom_third_deck_distance}" x_loc="0.09" y_loc="-0.165" z_loc="${eddie_plate_height}"/>
-  <robco_standoff parent="second_deck" subname="second_third_deck" number="2" lenght= "${top_second_botom_third_deck_distance}" x_loc="-0.09" y_loc="0.165" z_loc="${eddie_plate_height}"/>
-  <robco_standoff parent="second_deck" subname="second_third_deck" number="3" lenght= "${top_second_botom_third_deck_distance}" x_loc="-0.09" y_loc="-0.165" z_loc="${eddie_plate_height}"/>
+  <xacro:robco_standoff parent="second_deck" subname="second_third_deck" number="0" lenght= "${top_first_botom_second_deck_distance}" x_loc="0.09" y_loc="0.165" z_loc="${eddie_plate_height}"/>
+  <xacro:robco_standoff parent="second_deck" subname="second_third_deck" number="1" lenght= "${top_second_botom_third_deck_distance}" x_loc="0.09" y_loc="-0.165" z_loc="${eddie_plate_height}"/>
+  <xacro:robco_standoff parent="second_deck" subname="second_third_deck" number="2" lenght= "${top_second_botom_third_deck_distance}" x_loc="-0.09" y_loc="0.165" z_loc="${eddie_plate_height}"/>
+  <xacro:robco_standoff parent="second_deck" subname="second_third_deck" number="3" lenght= "${top_second_botom_third_deck_distance}" x_loc="-0.09" y_loc="-0.165" z_loc="${eddie_plate_height}"/>
 <!--########################################-->
 <!--######### THIRD DECK ###############################-->
@@ -632,9 +765,9 @@
     </collision>
     <visual name="third_deck__visual">
-      <!--<origin xyz="0 0 0" rpy="${ROTATE_90_DEGREES} 0 ${ROTATE_90_DEGREES}"/>-->
-       <origin xyz="0 0 0" rpy="0 0 0"/>
-      <geometry>
-        <cylinder radius="${base_radius}" length="${base_height}"/>
-        <!--<mesh filename="package://robot_description/meshes/Eddiebot/ArloBottomplateTST.dae" scale="0.001 0.001 0.001"/>-->
+       <!--<origin xyz="0 0 0" rpy="0 0 0"/>-->
+      <origin xyz="0 0 0" rpy="${ROTATE_90_DEGREES} 0 ${ROTATE_90_DEGREES}"/>
+      <geometry>
+        <!--<cylinder radius="${base_radius}" length="${base_height}"/>-->
+        <mesh filename="package://robot_description/meshes/Eddiebot/ArloBottomplateTST.dae" scale="0.001 0.001 0.001"/>
       </geometry>
       <material name="orange"/>
@@ -643,18 +776,15 @@
 <!--########################################-->
 <!--###########  KINECT STANDOFFS ON THIRD PLATE  #############################-->
-  <robco_standoff parent="third_deck" subname="third_deck_kinect" number="0" lenght= "${kinect_standoff_lenght-eddie_plate_height}" x_loc="${kinect_standoff_X_offset}" y_loc="${kinect_standoff_Y_offset}" z_loc="${kinect_standoff_Z_offset}"/>
-  <robco_standoff parent="third_deck" subname="third_deck_kinect" number="1" lenght= "${kinect_standoff_lenght-eddie_plate_height}" x_loc="${kinect_standoff_X_offset}" y_loc="${-kinect_standoff_Y_offset}" z_loc="${kinect_standoff_Z_offset}"/>
+  <xacro:robco_standoff parent="third_deck" subname="third_deck_kinect" number="0" lenght= "${kinect_standoff_lenght-eddie_plate_height}" x_loc="${kinect_standoff_X_offset}" y_loc="${kinect_standoff_Y_offset}" z_loc="${kinect_standoff_Z_offset}"/>
+  <xacro:robco_standoff parent="third_deck" subname="third_deck_kinect" number="1" lenght= "${kinect_standoff_lenght-eddie_plate_height}" x_loc="${kinect_standoff_X_offset}" y_loc="${-kinect_standoff_Y_offset}" z_loc="${kinect_standoff_Z_offset}"/>
   <!--<robco_standoff_kinect parent="third_deck" number="0"  x_loc="${kinect_mount_point_from_kinect_standoff_0__X_offset}" y_loc="0.06" z_loc="${eddie_plate_height}"/>
   <robco_standoff_kinect parent="third_deck" number="1"  x_loc="${kinect_mount_point_from_kinect_standoff_0__X_offset}" y_loc="-0.06" z_loc="${eddie_plate_height}"/>-->
 <!--###########  KINECT SUPPORT PLATE ON THE STANDOFFS  #############################-->
   <!--<robco_kinect_support_plate parent="standoff_third_deck_kinect_0_link" lenght= "${0.06}" width="${0.15}" height="${eddie_plate_height}" x_loc="${0.0}" y_loc="-0.06" z_loc="${(kinect_mount_point_from_kinect_standoff_0__Z_offset-eddie_plate_height)/2+eddie_plate_half_height}"/>-->
-  <robco_kinect_support_plate parent="standoff_third_deck_kinect_0_link" lenght= "${kinect_support_lenght}" width="${kinect_support_width}" height="${kinect_support_height}" x_loc="${kinect_support_from_kinect_standoff_0__X_offset}" y_loc="${kinect_support_from_kinect_standoff_0__Y_offset}" z_loc="${kinect_support_from_kinect_standoff_0__Z_offset}"/>
+  <xacro:robco_kinect_support_plate parent="standoff_third_deck_kinect_0_link" lenght= "${kinect_support_lenght}" width="${kinect_support_width}" height="${kinect_support_height}" x_loc="${kinect_support_from_kinect_standoff_0__X_offset}" y_loc="${kinect_support_from_kinect_standoff_0__Y_offset}" z_loc="${kinect_support_from_kinect_standoff_0__Z_offset}"/>
 <!--###########  KINECT MOUNT POINT ON THE KINECT SUPPORT PLATE  #############################-->
 <!--Visual for the kinect mount point comment out !!!!!!!!!!!!!!!!!!!!!!!!!!!!!!!!!!!!!!!!!!!!!!!!!!!!!!!!!!!!!!!!-->
-  <robco_mountpoint_visualizer_box parent="kinect_support_plate_link" device_name="kinect" lenght= "${0.005}" width="${0.005}" height="${0.005}" x_loc="${kinect_mount_point_from_support_plate_X_offset}" y_loc="${kinect_mount_point_from_support_plate_Y_offset}" z_loc="${kinect_mount_point_from_support_plate_Z_offset+kinect_support_height/2}"/>
-<!--########################################-->
-<!--###########  KINECT MOUNT POINT ON THE KINECT SUPPORT PLATE  #############################-->
-<!--Visual for the kinect mount point comment out !!!!!!!!!!!!!!!!!!!!!!!!!!!!!!!!!!!!!!!!!!!!!!!!!!!!!!!!!!!!!!!!-->
-  <!--<robco_mountpoint_visualizer_box parent="kinect_support_plate_link" device_name="kinect" lenght= "${0.005}" width="${0.005}" height="${0.005}" x_loc="${kinect_mount_point_from_support_plate_X_offset}" y_loc="${kinect_mount_point_from_support_plate_Y_offset}" z_loc="${kinect_mount_point_from_support_plate_Z_offset+kinect_support_height/2}"/>-->
+  <xacro:robco_mountpoint_visualizer_box parent="kinect_support_plate_link" device_name="kinect" lenght= "${0.005}" width="${0.005}" height="${0.005}" x_loc="${kinect_mount_point_from_support_plate_X_offset}" y_loc="${kinect_mount_point_from_support_plate_Y_offset}" z_loc="${kinect_mount_point_from_support_plate_Z_offset+kinect_support_height/2}"/>
+<!--The Joint to KINECT SUPPORT PLATE TO KINECT is already in the macro-->
  <!-- JOINT KINECT SUPPORT PLATE TO KINECT -->
   <!--<joint name="kinect_suppoet_plate_to_kinect_joint" type="fixed">
@@ -663,12 +793,16 @@
     <child link="kinect???????????????"/>
   </joint>-->
+  <!-- Attach the kinect_camera -->
+   <xacro:kinect_camera name="kinect_camera" parent="kinect_support_plate" color="Black">
+      <origin xyz="${0} ${0} ${kinect_support_height+kinect_support_half_height}" rpy="0 0 0" />
+   </xacro:kinect_camera>
 <!--########################################-->
 <!--###########  MOVER4 ARM MOUNT POINT ON THE KINECT SUPPORT PLATE  #############################-->
 <!--Visual for the kinect mount point comment out !!!!!!!!!!!!!!!!!!!!!!!!!!!!!!!!!!!!!!!!!!!!!!!!!!!!!!!!!!!!!!!!-->
- <mover4_arm/>
-  <robco_mountpoint_visualizer_box parent="third_deck" device_name="mover4_arm" lenght= "${eddie_plate_height}" width="${eddie_plate_height}" height="${eddie_plate_height}" x_loc="${0}" y_loc="${0}" z_loc="${eddie_plate_half_height+0.218}"/>
+ <xacro:mover4_arm/>
+  <xacro:robco_mountpoint_visualizer_box parent="third_deck" device_name="mover4_arm" lenght= "${eddie_plate_height}" width="${eddie_plate_height}" height="${eddie_plate_height}" x_loc="${0}" y_loc="${0}" z_loc="${eddie_plate_half_height+0.218}"/>
   <!--JOINT THIRD_DECK TO MOVER4_ARM -->
   <joint name="third_deck_mover4_arm_joint" type="fixed">
-    <origin rpy="0 0 1" xyz="0 0 ${eddie_plate_half_height}"/>
+    <origin rpy="0 0 0" xyz="${eddie_plate_radius-0.216} 0 ${eddie_plate_half_height}"/>
     <parent link="third_deck"/>
     <child link="arm_base_link"/>
@@ -695,5 +829,5 @@
     </inertial>
   </link>
-  <robco_mountpoint_visualizer_box parent="base_link" device_name="imu" lenght= "${0.05}" width="${0.05}" height="${0.05}" x_loc="${0.0}" y_loc="${0.0}" z_loc="${0.04}"/>
+  <xacro:robco_mountpoint_visualizer_box parent="base_link" device_name="imu" lenght= "${0.05}" width="${0.05}" height="${0.05}" x_loc="${0.0}" y_loc="${0.0}" z_loc="${0.04}"/>
 <!--########################################-->
 <!--######### LASER (RP Lidar) ###############################-->
@@ -708,5 +842,5 @@
         <box size="0.02 0.035 0.002" />
       </geometry>
-      <material name="Green" />
+      <material name="green" />
     </visual>
     <inertial>
@@ -718,6 +852,31 @@
     </inertial>
   </link>
-  <robco_mountpoint_visualizer_box parent="base_link" device_name="laser" lenght= "${0.05}" width="${0.05}" height="${0.05}" x_loc="${-0.065}" y_loc="${0.0}" z_loc="${0.075}"/>
-<!--########################################-->
+  <xacro:robco_mountpoint_visualizer_box parent="base_link" device_name="laser" lenght= "${0.05}" width="${0.05}" height="${0.05}" x_loc="${-0.065}" y_loc="${0.0}" z_loc="${0.075}"/>
+<!--########################################-->
+<!--######### TESTTTTTTTTTTTTTTTTTTTTTTTTTT ###############################-->
+  <joint name="test_joint" type="fixed">
+    <origin xyz="0.45 0 0.1" rpy="0 0 0" />
+    <parent link="base_link" />
+    <child link="test" />
+  </joint>
+  <link name="test">
+    <visual>
+      <geometry>
+        <!--<box size="0.02 0.035 0.002" />-->
+          <!--<mesh filename="package://robot_description/meshes/68-04556-RA_Kinect_Standoff_Assy.dae" scale="${SCALE_mm_m} ${SCALE_mm_m} ${SCALE_mm_m}"/>-->
+     <!--<mesh filename="package://robot_description/meshes/rplidar_a2/RPlidar_A2.stl.obj" scale="0.001 0.001 0.001"/>-->
+     <mesh filename="package://robot_description/meshes/Kinect/kinect.obj" scale="0 0 0"/>
+        <!--<box size="0.2 0.2 0.2" />-->
+      </geometry>
+      <!--<material name="green" />-->
+    </visual>
+    <inertial>
+      <mass value="0.001" />
+      <origin xyz="0 0 0" />
+      <inertia ixx="0.0001" ixy="0.0" ixz="0.0"
+        iyy="0.0001" iyz="0.0"
+        izz="0.0001" />
+    </inertial>
+  </link>
 <!--###########  KINECT  #############################-->
 <!--robco19_kinect_mount_point  standoff_third_deck_kinect_0_link-->
