Commit message: working on some meshes not displaying in RVIZ

File: robot_description/urdf/new_base.urdf.xacro (robot description, xacro)
@@ -832,13 +832,42 @@
 <!--########################################-->
 <!--######### LASER (RP Lidar) ###############################-->
+  <joint name="rplidar_joint" type="fixed">
+    <!--<axis xyz="0 1 0" />-->
+    <!--<origin xyz="0.02 0 0.086" rpy="0 0 0"/>-->
+    <origin xyz="0.50 0 ${eddie_plate_height+0.05}" rpy="0 0 0" />
+    <parent link="second_deck"/>
+    <child link="rplidar_laser_beam"/>
+  </joint>
+  <!-- rplidar Laser -->
+  <link name="rplidar_laser_beam">
+      <collision>
+      <origin xyz="0 0 0" rpy="0 0 0"/>
+      <geometry>
+        <box size="0.001 0.001 0.001"/>
+      </geometry>
+    </collision>
+   <visual>
+      <origin xyz="0 0 -0.03" rpy="1.5707 0 4.71"/>
+      <geometry>
+        <mesh filename="package://robot_description/meshes/rplidar-a2m4.stl" scale="0.001 0.001 0.001" />
+      </geometry>
+    </visual>
+    <inertial>
+      <mass value="1e-5" />
+      <origin xyz="0 0 0" rpy="0 0 0"/>
+      <inertia ixx="0" ixy="0" ixz="0" iyy="0" iyz="0" izz="0" />
+    </inertial>
+  </link>
   <joint name="laser_joint" type="fixed">
-    <origin xyz="-0.065 0 0.075" rpy="0 0 0" />
-    <parent link="base_link" />
-    <child link="laser" />
-  </joint>
-  <link name="laser">
+    <!--<origin xyz="-0.065 0 0.075" rpy="0 0 0" />-->
+    <origin xyz="0.20 0 ${eddie_plate_height}" rpy="0 0 0" />
+    <parent link="second_deck" />
+    <child link="laser_visual" />
+  </joint>
+  <link name="laser_visual">
     <visual>
       <geometry>
-        <box size="0.02 0.035 0.002" />
+     <mesh filename="package://robot_description/meshes/rplidar_a2/RPlidar_A2.stl.obj" scale="0.001 0.001 0.001"/>
+        <!--<box size="0.02 0.035 0.002" />-->
       </geometry>
       <material name="green" />
@@ -865,9 +894,10 @@
         <!--<box size="0.02 0.035 0.002" />-->
           <!--<mesh filename="package://robot_description/meshes/68-04556-RA_Kinect_Standoff_Assy.dae" scale="${SCALE_mm_m} ${SCALE_mm_m} ${SCALE_mm_m}"/>-->
+        	<!--<mesh filename="package://robot_description/meshes/GeometryCPRMover4/Joint0.obj" scale="0.001 0.001 0.001"/>-->
      <!--<mesh filename="package://robot_description/meshes/rplidar_a2/RPlidar_A2.stl.obj" scale="0.001 0.001 0.001"/>-->
-     <mesh filename="package://robot_description/meshes/Kinect/kinect.obj" scale="0 0 0"/>
+     <mesh filename="package://robot_description/meshes/kinect.dae.stl" scale="0.001 0.001 0.001"/>
         <!--<box size="0.2 0.2 0.2" />-->
       </geometry>
-      <!--<material name="green" />-->
+      <material name="red" />
     </visual>
     <inertial>
