Commit message: urdf cleanup, correct kinect frame orientation

File: robot_description/urdf/new_base.urdf.xacro (robot description, xacro)
@@ -17,5 +17,5 @@
 <!--###################################################################################-->
 <!--###################################################################################-->
-<!-- ####### generic constants ##### -->
+  <!-- ####### GENERIC CONSTANTS ##### -->
   <!--All units in m-kg-s-radians unit system -->
   <xacro:property name="PI" value="3.1415" />
@@ -25,48 +25,45 @@
   <xacro:property name="ROTATE_90_DEGREES" value="1.570796327" />
   <xacro:property name="DEG_TO_RAD" value="0.017453293" />
-  <xacro:property name="SCALE_in_m" value="0.0254"/> <!--inches to meters-->
-  <xacro:property name="SCALE_mm_m" value="0.001"/> <!--milimeters to meters-->
+  <xacro:property name="SCALE_in_to_m" value="0.0254"/> <!--inches to meters-->
+  <xacro:property name="SCALE_mm_to_m" value="0.001"/> <!--milimeters to meters-->
   <xacro:property name="kgcm_to_nm" value="0.0980665" />
-   <!-- ####### robot constants ##### -->
-  <xacro:property name="eddie_plate_height" value="${0.375*SCALE_in_m}" />
-  <xacro:property name="eddie_plate_half_height" value="${0.375*SCALE_in_m/2}" />
-  <xacro:property name="eddie_plate_diameter" value="${17.75*SCALE_in_m}" />
-  <xacro:property name="eddie_plate_radius" value="${17.75*SCALE_in_m/2}" />
-  <!-- base_link - Base Plate/Deck Cylinder base   -->
-  <xacro:property name="base_from_base_frame_Z_offset" value="${caster_assy_height}"/>   <!--da go naprawia param za macroto i ne triabva li da e +  eddie_plate_half_height  -->
-  <xacro:property name="base_height" value="${0.375*SCALE_in_m}" />
-  <xacro:property name="base_radius" value="${17.75*SCALE_in_m/2}" />
+  <!-- ####### ROBOT CONSTANTS ##### -->
+  <!--Baseframe to top of third deck height = 42.775 cm  ??? measure to confirm ???-->
+  <!-- ROUND PLATE DIMENSIONS  -->
+  <xacro:property name="round_plate_height" value="${0.375*SCALE_in_to_m}" />
+  <xacro:property name="round_plate_half_height" value="${0.375*SCALE_in_to_m/2}" />
+  <xacro:property name="round_plate_diameter" value="${17.75*SCALE_in_to_m}" />
+  <xacro:property name="round_plate_radius" value="${17.75*SCALE_in_to_m/2}" />
+  <!-- BASE PLATE   -->
+  <xacro:property name="base_plate_botom_from_base_frame_Z_offset" value="${caster_assy_height}"/>   <!--da go naprawia param za macroto i ne triabva li da e +  round_plate_half_height  -->
   <!-- in kg weight with the battery holder plate bellow -->
   <xacro:property name="base_mass" value="1.75" /> <!-- towa e tegloeoto samo na plochite, da dobavia egloto na akumulatorite dwigateliite i kolelata-->
-   <!-- distance between the robot origin and the bottom of the base plate along the z axis (robot up) -->
-  <!--<xacro:property name="BASE_PLATE_FROM_BASE_FRAME_Z_OFFSET" value="${caster_assy_height+eddie_plate_half_height}" />  meters -->
- <!-- second_deck - Base Plate/Deck Cylinder base   -->
+  <!-- SECOND DECK   -->
   <xacro:property name="top_first_botom_second_deck_distance" value="${0.145}" />
-  <xacro:property name="second_deck_from_base_link_Z_offset" value="${top_first_botom_second_deck_distance + eddie_plate_half_height}"/>
-  <xacro:property name="second_deck_height" value="${0.375*SCALE_in_m}" />
-  <xacro:property name="second_deck_radius" value="${17.75*SCALE_in_m/2}" />
+  <xacro:property name="second_deck_from_base_link_Z_offset" value="${top_first_botom_second_deck_distance + round_plate_half_height}"/>
+  <xacro:property name="second_deck_height" value="${0.375*SCALE_in_to_m}" />
+  <xacro:property name="second_deck_radius" value="${17.75*SCALE_in_to_m/2}" />
   <xacro:property name="second_deck_mass" value="1.5" />   <!-- in kg -->
-  <!-- third_deck - Base Plate/Deck Cylinder base   -->
+  <!-- THIRD DECK -->
   <xacro:property name="top_second_botom_third_deck_distance" value="${0.156}" />
-  <xacro:property name="third_deck_from_second_deck_Z_offset" value="${top_second_botom_third_deck_distance + eddie_plate_half_height}"/>
-  <xacro:property name="third_deck_height" value="${0.375*SCALE_in_m}" />
-  <xacro:property name="third_deck_radius" value="${17.75*SCALE_in_m/2}" />
+  <xacro:property name="third_deck_from_second_deck_Z_offset" value="${top_second_botom_third_deck_distance + round_plate_half_height}"/>
+  <xacro:property name="third_deck_height" value="${0.375*SCALE_in_to_m}" />
+  <xacro:property name="third_deck_radius" value="${17.75*SCALE_in_to_m/2}" />
   <xacro:property name="third_deck_mass" value="1.5" />   <!-- in kg -->
-<!--Base height to top of third deck = 42.775 cm ???-->
-  <!-- Wheels -->
-  <xacro:property name="wheel_diameter" value="${6*SCALE_in_m}" />
+  <!-- WHEELS -->
+  <xacro:property name="wheel_diameter" value="${6*SCALE_in_to_m}" />
   <xacro:property name="wheel_radius" value="${wheel_diameter/2}" />
-  <xacro:property name="wheel_width" value="${1.25*SCALE_in_m/2}" />
+  <xacro:property name="wheel_width" value="${1.25*SCALE_in_to_m/2}" />
   <xacro:property name="wheel_mass" value="0.6" /> <!-- ???? in kg-->
   <xacro:property name="base_x_origin_to_wheel_origin" value="0.0" />
   <xacro:property name="base_y_origin_to_wheel_origin" value="0.2" /> <!--VAJNO!!!!!! da se izmeri pak - ot tova zawisi odometriata!!!!!!!!!!! -->
     <!--<xacro:property name="base_y_origin_to_wheel_origin" value="0.19" />-->
-  <xacro:property name="base_z_origin_to_wheel_origin" value="${-(base_from_base_frame_Z_offset - wheel_radius)}" />
+  <xacro:property name="base_z_origin_to_wheel_origin" value="${-(base_plate_botom_from_base_frame_Z_offset - wheel_radius)}" />
+  <!-- CASTER WHEELS -->
   <!-- caster wheel offsets from base origin -->
   <xacro:property name="caster_X_offset_from_base_link" value="0.17"/>
-  <!-- caster wheel radius and height -->
-  <!-- caster wheel mass -->
+  <!-- caster wheel radius, height and mass -->
   <xacro:property name="caster_assy_height" value="${0.09825}" />
-  <xacro:property name="caster_wheel_radius" value="${3*SCALE_in_m/2}" />
+  <xacro:property name="caster_wheel_radius" value="${3*SCALE_in_to_m/2}" />
   <xacro:property name="caster_box_mass" value="0.15" /> <!-- in kg-->
   <xacro:property name="caster_box_height" value="${caster_assy_height- caster_wheel_radius*2}" />
@@ -76,37 +73,39 @@
   <xacro:property name="caster_sphere_diameter" value="${caster_wheel_radius*2}" />
   <xacro:property name="caster_sphere_radius" value="${caster_sphere_diameter/2}" />
+  <!-- STANDOFFS -->
+  <!-- deck standoff offsets -->
+  <xacro:property name="standoff_X_offset" value="${0.18 / 2}" />
+  <xacro:property name="standoff_Y_offset" value="${0.33 / 2}" />
   <!-- SENSORS -->
- <!-- Kinect -->
- <!-- kinect_mount_point - joint data for maunting kinect relative to base_link  -->
- <!--Kinect mount height 50 cm fro ground ?????-->
-    <xacro:property name="kinect_standoff_lenght" value="${0.42775}" />
-    <xacro:property name="kinect_standoff_X_offset" value="${-0.15}" />
-    <xacro:property name="kinect_standoff_Y_offset" value="${0.06}" />
-    <xacro:property name="kinect_standoff_Z_offset" value="${eddie_plate_height}" />
-  <!--<xacro:property name="kinect_mount_point_from_kinect_standoff_0__Z_offset" value="${(kinect_standoff_lenght - eddie_plate_height)/2+eddie_plate_height}" />
-  <xacro:property name="kinect_mount_point_from_kinect_standoff_0__X_offset" value="${0.15}"/>-->
+  <!-- KINECT -->
+  <xacro:property name="kinect_standoff_lenght" value="${0.42775}" /> <!-- ???????measure the real one???????????????-->
+  <xacro:property name="kinect_standoff_X_offset" value="${round_plate_radius-0.078}" />
+  <xacro:property name="kinect_standoff_Y_offset" value="${0.17 / 2}" />
+  <xacro:property name="kinect_standoff_Z_offset" value="${round_plate_height}" />
   <xacro:property name="kinect_mount_point_from_support_plate_X_offset" value="${0.0}"/>
   <xacro:property name="kinect_mount_point_from_support_plate_Y_offset" value="${0.0}" />
   <xacro:property name="kinect_mount_point_from_support_plate_Z_offset" value="${kinect_support_half_height}" />
   <xacro:property name="kinect_support_from_kinect_standoff_0__X_offset" value="${0.0}"/>
-  <xacro:property name="kinect_support_from_kinect_standoff_0__Y_offset" value="${-0.06}"/>
+  <xacro:property name="kinect_support_from_kinect_standoff_0__Y_offset" value="${-kinect_standoff_Y_offset}"/>
   <xacro:property name="kinect_support_from_kinect_standoff_0__Z_offset" value="${(kinect_standoff_lenght - kinect_support_height)/2+kinect_support_half_height}" />
-  <xacro:property name="kinect_support_height" value="${eddie_plate_height}" />
+  <xacro:property name="kinect_support_height" value="${round_plate_height}" />
   <xacro:property name="kinect_support_half_height" value="${kinect_support_height/2}" />
-  <xacro:property name="kinect_support_width" value="${0.15}" />
+  <xacro:property name="kinect_support_width" value="${kinect_standoff_Y_offset *2 + 0.05}" />
   <xacro:property name="kinect_support_lenght" value="${0.06}" />
   <xacro:property name="kinect_support_mass" value="${.05}" />    <!--in kg-->
-    <!-- Define a Kinect dimensions using properties -->
+    <!-- Define Kinect dimensions using properties -->
+   <xacro:property name="kinect_base_x" value="0.072" />
+   <xacro:property name="kinect_base_y" value="0.085" />
+   <xacro:property name="kinect_base_z" value="0.021" />
    <xacro:property name="kinect_body_x" value="0.07271" />
    <xacro:property name="kinect_body_y" value="0.27794" />
    <xacro:property name="kinect_body_z" value="0.033" />
-   <xacro:property name="kinect_base_x" value="0.072" />
-   <xacro:property name="kinect_base_y" value="0.085" />
-   <xacro:property name="kinect_base_z" value="0.021" />
    <xacro:property name="kinect_base_post_height" value="0.016" />
    <xacro:property name="kinect_base_post_radius" value="0.005" />
-  <!-- Hokuyo Laser scanner -->
-  <xacro:property name="hokuyo_size" value="${0.05}" />
-    <!-- camera -->
+  <!-- RPLIDAR A2  -->
+  <xacro:property name="rplidar_diameter" value="${0.0757}" />
+  <xacro:property name="rplidar_height_of_laser_beam_plane" value="${0.0308}" />
+  <xacro:property name="rplidar_height" value="${0.0408}" />
+    <!-- CAMERA -->
   <xacro:property name="cameraSize" value="${0.05}"/>
   <xacro:property name="cameraMass" value="${0.1}"/>
@@ -131,5 +130,5 @@
         <geometry>
           <cylinder length="${lenght}" radius="0.011113"/>
-          <!--<mesh filename="package://robot_description/meshes/68-02421-8000-RA_Eddiebot_F-F_Standoff.dae" scale="${SCALE_mm_m} ${SCALE_mm_m} ${SCALE_mm_m}"/>-->
+          <!--<mesh filename="package://robot_description/meshes/68-02421-8000-RA_Eddiebot_F-F_Standoff.dae" scale="${SCALE_mm_to_m} ${SCALE_mm_to_m} ${SCALE_mm_to_m}"/>-->
         </geometry>
         <material name="silver"/>
@@ -161,5 +160,5 @@
         <geometry>
           <cylinder length="${lenght}" radius="0.011113"/>
-          <!--<mesh filename="package://robot_description/meshes/68-02421-8000-RA_Eddiebot_F-F_Standoff.dae" scale="${SCALE_mm_m} ${SCALE_mm_m} ${SCALE_mm_m}"/>-->
+          <!--<mesh filename="package://robot_description/meshes/68-02421-8000-RA_Eddiebot_F-F_Standoff.dae" scale="${SCALE_mm_to_m} ${SCALE_mm_to_m} ${SCALE_mm_to_m}"/>-->
         </geometry>
         <material name="silver"/>
@@ -191,5 +190,5 @@
         <geometry>
           <cylinder length="${lenght}" radius="0.011113"/>
-          <!--<mesh filename="package://robot_description/meshes/68-02421-8000-RA_Eddiebot_F-F_Standoff.dae" scale="${SCALE_mm_m} ${SCALE_mm_m} ${SCALE_mm_m}"/>-->
+          <!--<mesh filename="package://robot_description/meshes/68-02421-8000-RA_Eddiebot_F-F_Standoff.dae" scale="${SCALE_mm_to_m} ${SCALE_mm_to_m} ${SCALE_mm_to_m}"/>-->
         </geometry>
         <material name="silver"/>
@@ -220,5 +219,5 @@
         <origin xyz=" 0 0 0 " rpy="0 0 0" />
         <geometry>
-          <mesh filename="package://robot_description/meshes/68-04556-RA_Kinect_Standoff_Assy.dae" scale="${SCALE_mm_m} ${SCALE_mm_m} ${SCALE_mm_m}"/>
+          <mesh filename="package://robot_description/meshes/68-04556-RA_Kinect_Standoff_Assy.dae" scale="${SCALE_mm_to_m} ${SCALE_mm_to_m} ${SCALE_mm_to_m}"/>
         </geometry>
       </visual>
@@ -249,5 +248,5 @@
         <geometry>
         <box size="${lenght} ${width} ${height}"/>
-          <!--<mesh filename="package://robot_description/meshes/68-02421-8000-RA_Eddiebot_F-F_Standoff.dae" scale="${SCALE_mm_m} ${SCALE_mm_m} ${SCALE_mm_m}"/>-->
+          <!--<mesh filename="package://robot_description/meshes/68-02421-8000-RA_Eddiebot_F-F_Standoff.dae" scale="${SCALE_mm_to_m} ${SCALE_mm_to_m} ${SCALE_mm_to_m}"/>-->
         </geometry>
         <material name="black"/>
@@ -279,5 +278,5 @@
         <geometry>
         <box size="${lenght} ${width} ${height}"/>
-          <!--<mesh filename="package://robot_description/meshes/68-02421-8000-RA_Eddiebot_F-F_Standoff.dae" scale="${SCALE_mm_m} ${SCALE_mm_m} ${SCALE_mm_m}"/>-->
+          <!--<mesh filename="package://robot_description/meshes/68-02421-8000-RA_Eddiebot_F-F_Standoff.dae" scale="${SCALE_mm_to_m} ${SCALE_mm_to_m} ${SCALE_mm_to_m}"/>-->
         </geometry>
         <material name="red"/>
@@ -357,5 +356,5 @@
       </link>
       <joint name="${name}_depth_joint" type="fixed">
-         <origin xyz="0 0.0125 0" rpy="0 0 0" />
+          <origin xyz="0 0.0125 0" rpy="0 0 0" />
           <parent link="${name}_link" />
           <child link="${name}_depth_frame" />
@@ -371,7 +370,8 @@
       </link>
       <joint name="${name}_depth_optical_joint" type="fixed">
-         <origin xyz="0 0 0" rpy="${-PI/2} 0 ${-PI/2}" />
-         <parent link="${name}_depth_frame" />
-         <child link="${name}_depth_optical_frame" />
+          <!--<origin xyz="0 0 0" rpy="${-M_PI_2} 0 ${-M_PI_2}" />-->
+          <origin xyz="0 0 0" rpy="${0} 0 ${0}" />
+          <parent link="${name}_depth_frame" />
+          <child link="${name}_depth_optical_frame" />
       </joint>
       <link name="${name}_depth_optical_frame">
@@ -399,5 +399,6 @@
       </link>
       <joint name="${name}_rgb_optical_joint" type="fixed">
-         <origin xyz="0 0 0" rpy="${-PI/2} 0 ${-PI/2}" />
+         <!--<origin xyz="0 0 0" rpy="${-M_PI_2} 0 ${-M_PI_2}" />-->
+         <origin xyz="0 0 0" rpy="${0} 0 ${0}" />
          <parent link="${name}_rgb_frame" />
          <child link="${name}_rgb_optical_frame" />
@@ -450,5 +451,5 @@
   <!-- JOINT BASE_LINK TO BASE_FRAME-->
   <joint name="base_footprint_base_link_joint" type="fixed">
-    <origin rpy="0 0 0" xyz="0 0 ${base_from_base_frame_Z_offset}"/>
+    <origin rpy="0 0 0" xyz="0 0 ${base_plate_botom_from_base_frame_Z_offset}"/>
     <parent link="base_footprint"/>
     <child link="base_link"/>
@@ -459,5 +460,5 @@
    <pose>0 0 0.1 0 0 0</pose>
    <inertial>
-      <origin xyz="0.0 0 ${eddie_plate_half_height}" rpy=" 0 0 0"/>
+      <origin xyz="0.0 0 ${round_plate_half_height}" rpy=" 0 0 0"/>
       <mass value="${base_mass}"/>
       <inertia
@@ -468,14 +469,14 @@
     </inertial>
     <collision name="collision">
-    <origin xyz="0 0 ${eddie_plate_half_height}" rpy="0 0 0" />
-      <geometry>
-       <cylinder radius="${eddie_plate_radius}" length="${eddie_plate_height}"/>
+    <origin xyz="0 0 ${round_plate_half_height}" rpy="0 0 0" />
+      <geometry>
+       <cylinder radius="${round_plate_radius}" length="${round_plate_height}"/>
       </geometry>
     </collision>
     <visual name="base_visual">
-      <!--<origin xyz="0 0 ${eddie_plate_half_height}" rpy="0 0 0" />      -->
+      <!--<origin xyz="0 0 ${round_plate_half_height}" rpy="0 0 0" />      -->
       <origin xyz="0 0 0" rpy="${ROTATE_90_DEGREES} 0 ${ROTATE_90_DEGREES}"/>
       <geometry>
-        <!--<cylinder radius="${eddie_plate_radius}" length="${eddie_plate_height}"/>-->
+        <!--<cylinder radius="${round_plate_radius}" length="${round_plate_height}"/>-->
         <mesh filename="package://robot_description/meshes/Eddiebot/ArloBottomplateTST.dae" scale="0.001 0.001 0.001"/>
       </geometry>
@@ -684,17 +685,17 @@
 <!--########################################-->
 <!--###########  STANDOFFS ON BASE PLATE  #############################-->
-  <!--<robco_standoff_first_second_deck parent="base_link" number="0" lenght= "${top_first_botom_second_deck_distance}" x_loc="0.09" y_loc="0.165" z_loc="${eddie_plate_height}"/>
-  <robco_standoff_first_second_deck parent="base_link" number="1" lenght= "${top_first_botom_second_deck_distance}" x_loc="0.09" y_loc="-0.165" z_loc="${eddie_plate_height}"/>
-  <robco_standoff_first_second_deck parent="base_link" number="2" lenght= "${top_first_botom_second_deck_distance}" x_loc="-0.09" y_loc="0.165" z_loc="${eddie_plate_height}"/>
-  <robco_standoff_first_second_deck parent="base_link" number="3" lenght= "${top_first_botom_second_deck_distance}" x_loc="-0.09" y_loc="-0.165" z_loc="${eddie_plate_height}"/>-->
-  <xacro:robco_standoff parent="base_link" subname="first_second_deck" number="0" lenght= "${top_first_botom_second_deck_distance}" x_loc="0.09" y_loc="0.165" z_loc="${eddie_plate_height}"/>
-  <xacro:robco_standoff parent="base_link" subname="first_second_deck" number="1" lenght= "${top_first_botom_second_deck_distance}" x_loc="0.09" y_loc="-0.165" z_loc="${eddie_plate_height}"/>
-  <xacro:robco_standoff parent="base_link" subname="first_second_deck" number="2" lenght= "${top_first_botom_second_deck_distance}" x_loc="-0.09" y_loc="0.165" z_loc="${eddie_plate_height}"/>
-  <xacro:robco_standoff parent="base_link" subname="first_second_deck" number="3" lenght= "${top_first_botom_second_deck_distance}" x_loc="-0.09" y_loc="-0.165" z_loc="${eddie_plate_height}"/>
+  <!--<robco_standoff_first_second_deck parent="base_link" number="0" lenght= "${top_first_botom_second_deck_distance}" x_loc="0.09" y_loc="0.165" z_loc="${round_plate_height}"/>
+  <robco_standoff_first_second_deck parent="base_link" number="1" lenght= "${top_first_botom_second_deck_distance}" x_loc="0.09" y_loc="-0.165" z_loc="${round_plate_height}"/>
+  <robco_standoff_first_second_deck parent="base_link" number="2" lenght= "${top_first_botom_second_deck_distance}" x_loc="-0.09" y_loc="0.165" z_loc="${round_plate_height}"/>
+  <robco_standoff_first_second_deck parent="base_link" number="3" lenght= "${top_first_botom_second_deck_distance}" x_loc="-0.09" y_loc="-0.165" z_loc="${round_plate_height}"/>-->
+  <xacro:robco_standoff parent="base_link" subname="first_second_deck" number="0" lenght= "${top_first_botom_second_deck_distance}" x_loc="${standoff_X_offset}" y_loc="${standoff_Y_offset}" z_loc="${round_plate_height}"/>
+  <xacro:robco_standoff parent="base_link" subname="first_second_deck" number="1" lenght= "${top_first_botom_second_deck_distance}" x_loc="${standoff_X_offset}" y_loc="${-standoff_Y_offset}" z_loc="${round_plate_height}"/>
+  <xacro:robco_standoff parent="base_link" subname="first_second_deck" number="2" lenght= "${top_first_botom_second_deck_distance}" x_loc="${-standoff_X_offset}" y_loc="${standoff_Y_offset}" z_loc="${round_plate_height}"/>
+  <xacro:robco_standoff parent="base_link" subname="first_second_deck" number="3" lenght= "${top_first_botom_second_deck_distance}" x_loc="${-standoff_X_offset}" y_loc="${-standoff_Y_offset}" z_loc="${round_plate_height}"/>
 <!--########################################-->
 <!--###########  SECOND DECK  #############################-->
  <!-- JOINT second_deck TO BASE_LINK -->
   <joint name="base_link_second_deck_joint" type="fixed">
-    <origin rpy="0 0 0" xyz="0 0 ${second_deck_from_base_link_Z_offset+eddie_plate_half_height}"/>
+    <origin rpy="0 0 0" xyz="0 0 ${second_deck_from_base_link_Z_offset+round_plate_half_height}"/>
     <parent link="base_link"/>
     <child link="second_deck"/>
@@ -713,14 +714,14 @@
     </inertial>
     <collision name="collision">
-        <origin xyz="0 0 ${eddie_plate_half_height}" rpy="0 0 0" />
-      <geometry>
-       <cylinder radius="${eddie_plate_radius}" length="${eddie_plate_height}"/>
+        <origin xyz="0 0 ${round_plate_half_height}" rpy="0 0 0" />
+      <geometry>
+       <cylinder radius="${round_plate_radius}" length="${round_plate_height}"/>
       </geometry>
     </collision>
     <visual name="second_deck_visual">
-        <!--<origin xyz="0 0 ${eddie_plate_half_height}" rpy="0 0 0" />      -->
+        <!--<origin xyz="0 0 ${round_plate_half_height}" rpy="0 0 0" />      -->
       <origin xyz="0 0 0" rpy="${ROTATE_90_DEGREES} 0 ${ROTATE_90_DEGREES}"/>
       <geometry>
-        <!--<cylinder radius="${eddie_plate_radius}" length="${eddie_plate_height}"/>-->
+        <!--<cylinder radius="${round_plate_radius}" length="${round_plate_height}"/>-->
         <mesh filename="package://robot_description/meshes/Eddiebot/ArloBottomplateTST.dae" scale="0.001 0.001 0.001"/>
       </geometry>
@@ -730,17 +731,17 @@
 <!--########################################-->
 <!--###########  STANDOFFS ON SECOND PLATE  #############################-->
-  <!--<robco_standoff parent="second_deck" subname="second_third_deck" number="0" lenght= "${top_first_botom_second_deck_distance}" x_loc="0.09" y_loc="0.165" z_loc="${eddie_plate_height}"/>
-  <robco_standoff_second_third_deck parent="second_deck" number="1" lenght= "${top_second_botom_third_deck_distance}" x_loc="0.09" y_loc="-0.165" z_loc="${eddie_plate_height}"/>
-  <robco_standoff_second_third_deck parent="second_deck" number="2" lenght= "${top_second_botom_third_deck_distance}" x_loc="-0.09" y_loc="0.165" z_loc="${eddie_plate_height}"/>
-  <robco_standoff_second_third_deck parent="second_deck" number="3" lenght= "${top_second_botom_third_deck_distance}" x_loc="-0.09" y_loc="-0.165" z_loc="${eddie_plate_height}"/>-->
-  <xacro:robco_standoff parent="second_deck" subname="second_third_deck" number="0" lenght= "${top_first_botom_second_deck_distance}" x_loc="0.09" y_loc="0.165" z_loc="${eddie_plate_height}"/>
-  <xacro:robco_standoff parent="second_deck" subname="second_third_deck" number="1" lenght= "${top_second_botom_third_deck_distance}" x_loc="0.09" y_loc="-0.165" z_loc="${eddie_plate_height}"/>
-  <xacro:robco_standoff parent="second_deck" subname="second_third_deck" number="2" lenght= "${top_second_botom_third_deck_distance}" x_loc="-0.09" y_loc="0.165" z_loc="${eddie_plate_height}"/>
-  <xacro:robco_standoff parent="second_deck" subname="second_third_deck" number="3" lenght= "${top_second_botom_third_deck_distance}" x_loc="-0.09" y_loc="-0.165" z_loc="${eddie_plate_height}"/>
+  <!--<robco_standoff parent="second_deck" subname="second_third_deck" number="0" lenght= "${top_first_botom_second_deck_distance}" x_loc="0.09" y_loc="0.165" z_loc="${round_plate_height}"/>
+  <robco_standoff_second_third_deck parent="second_deck" number="1" lenght= "${top_second_botom_third_deck_distance}" x_loc="0.09" y_loc="-0.165" z_loc="${round_plate_height}"/>
+  <robco_standoff_second_third_deck parent="second_deck" number="2" lenght= "${top_second_botom_third_deck_distance}" x_loc="-0.09" y_loc="0.165" z_loc="${round_plate_height}"/>
+  <robco_standoff_second_third_deck parent="second_deck" number="3" lenght= "${top_second_botom_third_deck_distance}" x_loc="-0.09" y_loc="-0.165" z_loc="${round_plate_height}"/>-->
+  <xacro:robco_standoff parent="second_deck" subname="second_third_deck" number="0" lenght= "${top_second_botom_third_deck_distance}" x_loc="${standoff_X_offset}" y_loc="${standoff_Y_offset}" z_loc="${round_plate_height}"/>
+  <xacro:robco_standoff parent="second_deck" subname="second_third_deck" number="1" lenght= "${top_second_botom_third_deck_distance}" x_loc="${standoff_X_offset}" y_loc="${-standoff_Y_offset}" z_loc="${round_plate_height}"/>
+  <xacro:robco_standoff parent="second_deck" subname="second_third_deck" number="2" lenght= "${top_second_botom_third_deck_distance}" x_loc="${-standoff_X_offset}" y_loc="${standoff_Y_offset}" z_loc="${round_plate_height}"/>
+  <xacro:robco_standoff parent="second_deck" subname="second_third_deck" number="3" lenght= "${top_second_botom_third_deck_distance}" x_loc="${-standoff_X_offset}" y_loc="${-standoff_Y_offset}" z_loc="${round_plate_height}"/>
 <!--########################################-->
 <!--######### THIRD DECK ###############################-->
   <!-- JOINT THIRD_DECK TO SECOND_DECK -->
   <joint name="third_deck_second_deck_joint" type="fixed">
-    <origin rpy="0 0 0" xyz="0 0 ${third_deck_from_second_deck_Z_offset+eddie_plate_half_height}"/>
+    <origin rpy="0 0 0" xyz="0 0 ${third_deck_from_second_deck_Z_offset+round_plate_half_height}"/>
     <parent link="second_deck"/>
     <child link="third_deck"/>
@@ -759,7 +760,7 @@
     </inertial>
     <collision name="collision">
-      <origin xyz="0 0 ${eddie_plate_half_height}" rpy="0 0 0" />
-      <geometry>
-       <cylinder radius="${eddie_plate_radius}" length="${eddie_plate_height}"/>
+      <origin xyz="0 0 ${round_plate_half_height}" rpy="0 0 0" />
+      <geometry>
+       <cylinder radius="${round_plate_radius}" length="${round_plate_height}"/>
       </geometry>
     </collision>
@@ -768,5 +769,4 @@
       <origin xyz="0 0 0" rpy="${ROTATE_90_DEGREES} 0 ${ROTATE_90_DEGREES}"/>
       <geometry>
-        <!--<cylinder radius="${base_radius}" length="${base_height}"/>-->
         <mesh filename="package://robot_description/meshes/Eddiebot/ArloBottomplateTST.dae" scale="0.001 0.001 0.001"/>
       </geometry>
@@ -776,10 +776,10 @@
 <!--########################################-->
 <!--###########  KINECT STANDOFFS ON THIRD PLATE  #############################-->
-  <xacro:robco_standoff parent="third_deck" subname="third_deck_kinect" number="0" lenght= "${kinect_standoff_lenght-eddie_plate_height}" x_loc="${kinect_standoff_X_offset}" y_loc="${kinect_standoff_Y_offset}" z_loc="${kinect_standoff_Z_offset}"/>
-  <xacro:robco_standoff parent="third_deck" subname="third_deck_kinect" number="1" lenght= "${kinect_standoff_lenght-eddie_plate_height}" x_loc="${kinect_standoff_X_offset}" y_loc="${-kinect_standoff_Y_offset}" z_loc="${kinect_standoff_Z_offset}"/>
-  <!--<robco_standoff_kinect parent="third_deck" number="0"  x_loc="${kinect_mount_point_from_kinect_standoff_0__X_offset}" y_loc="0.06" z_loc="${eddie_plate_height}"/>
-  <robco_standoff_kinect parent="third_deck" number="1"  x_loc="${kinect_mount_point_from_kinect_standoff_0__X_offset}" y_loc="-0.06" z_loc="${eddie_plate_height}"/>-->
+  <xacro:robco_standoff parent="third_deck" subname="third_deck_kinect" number="0" lenght= "${kinect_standoff_lenght-round_plate_height}" x_loc="${-kinect_standoff_X_offset}" y_loc="${kinect_standoff_Y_offset}" z_loc="${kinect_standoff_Z_offset}"/>
+  <xacro:robco_standoff parent="third_deck" subname="third_deck_kinect" number="1" lenght= "${kinect_standoff_lenght-round_plate_height}" x_loc="${-kinect_standoff_X_offset}" y_loc="${-kinect_standoff_Y_offset}" z_loc="${kinect_standoff_Z_offset}"/>
+  <!--<robco_standoff_kinect parent="third_deck" number="0"  x_loc="${kinect_mount_point_from_kinect_standoff_0__X_offset}" y_loc="0.06" z_loc="${round_plate_height}"/>
+  <robco_standoff_kinect parent="third_deck" number="1"  x_loc="${kinect_mount_point_from_kinect_standoff_0__X_offset}" y_loc="-0.06" z_loc="${round_plate_height}"/>-->
 <!--###########  KINECT SUPPORT PLATE ON THE STANDOFFS  #############################-->
-  <!--<robco_kinect_support_plate parent="standoff_third_deck_kinect_0_link" lenght= "${0.06}" width="${0.15}" height="${eddie_plate_height}" x_loc="${0.0}" y_loc="-0.06" z_loc="${(kinect_mount_point_from_kinect_standoff_0__Z_offset-eddie_plate_height)/2+eddie_plate_half_height}"/>-->
+  <!--<robco_kinect_support_plate parent="standoff_third_deck_kinect_0_link" lenght= "${0.06}" width="${0.15}" height="${round_plate_height}" x_loc="${0.0}" y_loc="-0.06" z_loc="${(kinect_mount_point_from_kinect_standoff_0__Z_offset-round_plate_height)/2+round_plate_half_height}"/>-->
   <xacro:robco_kinect_support_plate parent="standoff_third_deck_kinect_0_link" lenght= "${kinect_support_lenght}" width="${kinect_support_width}" height="${kinect_support_height}" x_loc="${kinect_support_from_kinect_standoff_0__X_offset}" y_loc="${kinect_support_from_kinect_standoff_0__Y_offset}" z_loc="${kinect_support_from_kinect_standoff_0__Z_offset}"/>
 <!--###########  KINECT MOUNT POINT ON THE KINECT SUPPORT PLATE  #############################-->
@@ -789,5 +789,5 @@
  <!-- JOINT KINECT SUPPORT PLATE TO KINECT -->
   <!--<joint name="kinect_suppoet_plate_to_kinect_joint" type="fixed">
-    <origin rpy="0 0 0" xyz="0 0 ${third_deck_from_second_deck_Z_offset+eddie_plate_half_height}"/>
+    <origin rpy="0 0 0" xyz="0 0 ${third_deck_from_second_deck_Z_offset+round_plate_half_height}"/>
     <parent link="kinect_support_plate_link"/>
     <child link="kinect???????????????"/>
@@ -801,8 +801,8 @@
 <!--Visual for the kinect mount point comment out !!!!!!!!!!!!!!!!!!!!!!!!!!!!!!!!!!!!!!!!!!!!!!!!!!!!!!!!!!!!!!!!-->
  <xacro:mover4_arm/>
-  <xacro:robco_mountpoint_visualizer_box parent="third_deck" device_name="mover4_arm" lenght= "${eddie_plate_height}" width="${eddie_plate_height}" height="${eddie_plate_height}" x_loc="${0}" y_loc="${0}" z_loc="${eddie_plate_half_height+0.218}"/>
+  <xacro:robco_mountpoint_visualizer_box parent="third_deck" device_name="mover4_arm" lenght= "${round_plate_height}" width="${round_plate_height}" height="${round_plate_height}" x_loc="${0}" y_loc="${0}" z_loc="${round_plate_half_height+0.218}"/>
   <!--JOINT THIRD_DECK TO MOVER4_ARM -->
   <joint name="third_deck_mover4_arm_joint" type="fixed">
-    <origin rpy="0 0 0" xyz="${eddie_plate_radius-0.216} 0 ${eddie_plate_half_height}"/>
+    <origin rpy="0 0 0" xyz="${round_plate_radius-0.216} 0 ${round_plate_half_height}"/>
     <parent link="third_deck"/>
     <child link="arm_base_link"/>
@@ -829,5 +829,5 @@
     </inertial>
   </link>
-  <xacro:robco_mountpoint_visualizer_box parent="base_link" device_name="imu" lenght= "${0.05}" width="${0.05}" height="${0.05}" x_loc="${0.0}" y_loc="${0.0}" z_loc="${0.04}"/>
+  <xacro:robco_mountpoint_visualizer_box parent="base_link" device_name="imu" lenght= "${0.01}" width="${0.01}" height="${0.01}" x_loc="${0.0}" y_loc="${0.0}" z_loc="${0.04}"/>
 <!--########################################-->
 <!--######### LASER (RP Lidar) ###############################-->
@@ -835,21 +835,25 @@
     <!--<axis xyz="0 1 0" />-->
     <!--<origin xyz="0.02 0 0.086" rpy="0 0 0"/>-->
-    <origin xyz="0.50 0 ${eddie_plate_height+0.05}" rpy="0 0 0" />
+    <origin xyz="${round_plate_radius-rplidar_diameter/2-0.01} 0 ${round_plate_height+rplidar_height_of_laser_beam_plane}" rpy="0 0 0" />
     <parent link="second_deck"/>
-    <child link="rplidar_laser_beam"/>
+    <child link="rplidar_laser_beam_plane"/>
   </joint>
   <!-- rplidar Laser -->
-  <link name="rplidar_laser_beam">
+  <link name="rplidar_laser_beam_plane">
       <collision>
       <origin xyz="0 0 0" rpy="0 0 0"/>
       <geometry>
-        <box size="0.001 0.001 0.001"/>
-      </geometry>
+        <cylinder length="0.01" radius="0.2"/>
+      </geometry>
+      <material name="green" />
     </collision>
-   <visual>
-      <origin xyz="0 0 -0.03" rpy="1.5707 0 4.71"/>
-      <geometry>
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